File: Puck.kicad_sch (KiCad schematic)
At the start: 22 parts

Commit message: WIP
Parts:
- added C4: 1uF, 35V, Capacitor_SMD:C_0603_1608Metric_Pad1.08x0.95mm_HandSolder, symbol Device:C
- added D3, D4: LED, LED_SMD:LED_0603_1608Metric_Pad1.05x0.95mm_HandSolder, symbol Device:LED
- added TP1: TestPoint, TestPoint:TestPoint_Pad_2.0x2.0mm, symbol Connector:TestPoint
- C1, C2, C3: renamed from C?; value C -> 0.1uF; footprint (none) -> Capacitor_SMD:C_0603_1608Metric_Pad1.08x0.95mm_HandSolder
- D2: renamed from D?; footprint (none) -> LED_SMD:LED_0603_1608Metric_Pad1.05x0.95mm_HandSolder
- Q1: renamed from Q?; footprint (none) -> Package_TO_SOT_SMD:SOT-23
- R1, R2, R4, R5: renamed from R?; value R -> 10K; footprint (none) -> Resistor_SMD:R_0603_1608Metric_Pad0.98x0.95mm_HandSolder
- R3: renamed from R?; value R -> 82K; footprint (none) -> Resistor_SMD:R_0603_1608Metric_Pad0.98x0.95mm_HandSolder
- R6, R7: renamed from R?; footprint (none) -> Resistor_SMD:R_0603_1608Metric_Pad0.98x0.95mm_HandSolder
- R8: renamed from R?; value R -> 1K; footprint (none) -> Resistor_SMD:R_0603_1608Metric_Pad0.98x0.95mm_HandSolder
- RV1: renamed from RV?; value R_Potentiometer -> 1M; footprint (none) -> Potentiometer_SMD:Potentiometer_Bourns_3314J_Vertical
- RV2: renamed from RV?; value R_Potentiometer -> 100K; footprint (none) -> Potentiometer_SMD:Potentiometer_Bourns_3314J_Vertical
- U1: renamed from U?; value TLC274 -> LM324PT; footprint (none) -> Package_SO:TSSOP-14_4.4x5mm_P0.65mm; symbol Amplifier_Operational:TLC274 -> Amplifier_Operational:LM324
- gave numbers to parts that had none: 1
Connections:
- net GND: now also C4.1, D4.1 (K); no longer D2.1 (K)
- net PZ+: now also TP1.1
- net VCC: now also C4.2
- net OUT: no longer names the net of Q1.2 (C)
- new net: D2.1 (K), D3.2 (A)
- new net: D3.1 (K), D4.2 (A)
Other:
- moved on the sheet: C1, C2, C3, D1A, D1B, D2, Q1, R1, R2, R3, R4, R5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
